File: hardware/powerdist-hw.brd (EAGLE design)
At the start: 100 x 18 mm, 31 parts, among them IC1 AVRXDA32TQFP, IC3 ACS712, Q1 NFET SO8, Q2 NFET SO8, Q3 NFET SO8, Q4 NFET SO8, Q5 NFET SO8

Commit message: lots of progress
Parts:
- added C5: 100n, rcl:C0603
- added J1: (no value), SparkFun-Connectors:JST-5-PTH
- added R10, R6, R8: 10K, rcl:R0603
- added R7: (no value), rcl:R0603
- added R9: 100R, SparkFun-Resistors:0603-ARV
- added RDIV10, RDIV9: 50K, SparkFun-Resistors:0805
- added UPDI: (no value), SparkFun-Connectors:1X03
- C1: value 1u -> 100n; device SparkFun-Passives:0805 -> rcl:C0603
- C2: device SparkFun-Passives:0805 -> rcl:C0805
- C3, C4: device SparkFun-Passives:0603-CAP -> rcl:C0603
- IC2: device v-reg:SOT23 -> v-reg:78XXS
- Q1, Q2, Q3, Q4: value NFET SO8 -> (none); device SparkFun-DiscreteSemi:SO08 -> transistor-generic:SO-08
- R1, R2, R3, R4, R5: device SparkFun-Resistors:0603-RES -> rcl:R0603
- moved R1 22.2 mm to (26.7, 3.81), turned to 270 degrees
- moved VR1 21.0 mm to (30.5, 3.81)
- moved R2 18.8 mm to (34.3, 15.2), turned to 90 degrees
- moved C1 18.5 mm to (24.4, 3.81)
- moved R3 17.4 mm to (44.8, 15.2), turned to 90 degrees
- moved R4 16.3 mm to (54.9, 15.2), turned to 90 degrees
- moved R5 14.2 mm to (65.1, 15.2), turned to 90 degrees
- moved IC3 14.0 mm to (74.3, 8.89), turned to 0 degrees
- moved OUT 13.2 mm to (78.5, 3.17), turned to 180 degrees
- moved RDIV5 12.0 mm to (30.5, 15.2), turned to 270 degrees
- moved RDIV1 9.52 mm to (32.4, 15.2)
- moved RDIV6 7.96 mm to (42.9, 12.1)
- moved RDIV2 7.94 mm to (42.9, 15.2)
- moved C3 7.65 mm to (25.4, 6.99)
- moved BAT1 7.62 mm to (39.4, 15.2)
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Connections:
- new net GATE1: Q1.4, R2.1, R9.4
- new net GATE1`: IC1.25, R9.5
- new net GATE2: Q2.4, R3.1, R9.3
- new net GATE3: Q3.4, R4.1, R9.2
- new net GATE4: Q4.4, R5.1, R9.1
- new net GATE5: Q5.4, R6.2, R7.2
- new net GATE5`: IC1.21, R7.1
- new net N$1: IC3.7, RDIV9.2
- new net N$2: IC1.27, UPDI.2
- new net N$3: IC1.22, R9.8
- new net N$4: IC1.23, R9.7
- new net N$5: IC1.24, R9.6
- new net SCL: IC1.1, R10.1
- new net SDA: IC1.32, R8.1
- new net VLOAD: IC1.14, RDIV10.2, RDIV9.1
- net +12V: no longer C1.1, IC2.3
- net AREF: now also C1.1
- net BAT1+: now also IC2.IN, R2.2
- net BAT2+: now also R3.2
- net BAT3+: now also R4.2
- net BAT4+: now also R5.2
- net GND: now also C5.2, IC2.GND, IC3.5, J1.1, J1.3, R6.1, RDIV10.1, UPDI.1
- net VCC: now also C5.1, IC2.OUT, IC3.8, R10.2, R8.2, UPDI.3; no longer IC2.2
Routing:
- net VLOAD: track 0.00 -> 69.6 mm, vias 0 -> 2
- net GATE5`: track 0.00 -> 63.7 mm, vias 0 -> 2
- net VBAT4: track 0.00 -> 52.0 mm, vias 0 -> 2
- net GATE4: track 0.00 -> 47.4 mm
- net VBAT3: track 0.00 -> 42.4 mm, vias 0 -> 2
- net GATE3: track 0.00 -> 37.5 mm
- net VCC: track 0.00 -> 36.2 mm, vias 0 -> 1
- net VBAT2: track 0.00 -> 33.4 mm, vias 0 -> 2
- net GATE2: track 0.00 -> 26.6 mm
- net VBAT1: track 0.00 -> 23.1 mm, vias 0 -> 2
- net GATE1: track 0.00 -> 13.1 mm
- net AREF: track 0.00 -> 11.2 mm
- net GATE5: track 0.00 -> 6.06 mm
- net SCL: track 0.00 -> 5.40 mm
- net GATE1`: track 0.00 -> 4.54 mm
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- added copper zone on layer 1, net +12V
- added copper zone on layer 16, net GND
Other:
- board size 100 x 18 mm -> 84.8 x 18 mm

Commit message: layout complete
Parts:
- moved VR1 2.01 mm to (32.4, 4.45)
- moved BAT4 1.31 mm to (71.1, 14.9)
- moved RDIV10 1.31 mm to (77.2, 14.9)
- moved BAT1 1.31 mm to (40.6, 14.9)
- moved BAT3 1.31 mm to (61.0, 14.9)
- moved Q2 1.31 mm to (49.5, 8.57)
- moved R2 1.31 mm to (35.6, 14.9)
- moved R3 1.31 mm to (46.0, 14.9)
- moved RDIV1 1.31 mm to (33.7, 14.9)
- moved RDIV2 1.31 mm to (44.1, 14.9)
- moved RDIV4 1.31 mm to (64.5, 14.9)
- moved RDIV6 1.31 mm to (44.1, 11.7)
- moved RDIV8 1.31 mm to (64.5, 11.7)
- moved RDIV5 1.31 mm to (31.8, 14.9)
- moved BAT2 1.31 mm to (50.8, 14.9)
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Connections:
- net SCL: now also J1.2
- net SDA: now also J1.4
- net VCC: now also J1.5
Routing:
- net VCC: track 36.2 -> 128.8 mm, vias 1 -> 4
- net BAT1+: track 6.12 -> 36.2 mm
- net SCL: track 5.40 -> 15.9 mm
- net SDA: track 4.48 -> 14.0 mm, vias 0 -> 1
- net N$2: track 0.00 -> 5.77 mm
- net VLOAD: track 69.6 -> 71.5 mm
- net GATE2: track 26.6 -> 27.8 mm
Other:
- board size 84.8 x 18 mm -> 86 x 18 mm
