File: hardware/powerdist-hw.sch (EAGLE design)
At the start: 31 parts, among them IC1 AVRXDA32TQFP, IC3 ACS712, Q1 NFET SO8, Q2 NFET SO8, Q3 NFET SO8, Q4 NFET SO8, Q5 NFET SO8

Commit message: lots of progress
Parts:
- added C5: 100n, rcl:C-EUC0603
- added J1: (no value), SparkFun-Connectors:M05JST
- added R10, R6, R8: 10K, rcl:R-US_R0603
- added R7: (no value), rcl:R-US_R0603
- added R9: 100R, SparkFun-Resistors:RESISTOR-ARRAY0603-ARV
- added RDIV10, RDIV9: 50K, SparkFun-Resistors:RESISTOR0805-RES
- added UPDI: (no value), SparkFun-Connectors:M03PTH
- C1: value 1u -> 100n; device SparkFun-Passives:CAP0805 -> rcl:C-EUC0603
- C2: device SparkFun-Passives:CAP0805 -> rcl:C-USC0805
- C3, C4: device SparkFun-Passives:CAP0603-CAP -> rcl:C-EUC0603
- IC2: device v-reg:XC63FPM -> v-reg:78XXS
- Q1, Q2, Q3, Q4: value NFET SO8 -> (none); device SparkFun-DiscreteSemi:MOSFET-NCHANNELFDS6630A -> transistor-generic:PFETSO8
- R1, R2, R3, R4, R5: device SparkFun-Resistors:RESISTOR0603-RES -> rcl:R-US_R0603
Connections:
- new net GATE1: Q1.G, R2.1, R9D.1
- new net GATE1`: IC1.PF5(AIN21/RXD2), R9D.2
- new net GATE2: Q2.G, R3.1, R9C.1
- new net GATE3: Q3.G, R4.1, R9B.1
- new net GATE4: Q4.G, R5.1, R9A.1
- new net GATE5: Q5.G, R6.2, R7.2
- new net GATE5`: IC1.PF1(AIN17/RXD2/3IN1/TOSC2), R7.1
- new net N$1: IC3.VOUT, RDIV9.2
- new net N$2: IC1.UPDI, UPDI.2
- new net N$3: IC1.PF2(SDA1/AIN18/3-IN2), R9A.2
- new net N$4: IC1.PF3(SCL1/AIN19/3-OUT), R9B.2
- new net N$5: IC1.PF4(AIN20/TXD2), R9C.2
- new net SCL: IC1.PA3(SCL0/0-OUT/TCB1), R10.1
- new net SDA: IC1.PA2(SDA0/0-IN2/TCBO), R8.1
- new net VLOAD: IC1.PD4(A4/AIN4/AC-P1/TCA0), RDIV10.2, RDIV9.1
- net +12V: no longer C1.1, IC2.IN
- net AREF: now also C1.1
- net BAT1+: now also IC2.IN, R2.2
- net BAT2+: now also R3.2
- net BAT3+: now also R4.2
- net BAT4+: now also R5.2
- net GND: now also C5.2, IC2.GND, IC3.GND, J1.1, J1.3, R6.1, RDIV10.1, UPDI.1
- net VCC: now also C5.1, IC3.VCC, R10.2, R8.2, UPDI.3
Other:
- moved on the sheet: C1, C2, C3, C4, R2, R3, R4, R5, RDIV1, RDIV2, RDIV3, RDIV4

Commit message: layout complete
Connections:
- net SCL: now also J1.2
- net SDA: now also J1.4
- net VCC: now also J1.5
Changed lines of the file:
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@@
 <grid distance="0.1" unitdist="inch" unit="inch" style="lines" multiple="1" display="no" altdistance="0.01" altunitdist="inch" altunit="inch"/>
 <layers>
-<layer number="1" name="Top" color="4" fill="1" visible="yes" active="no"/>
-<layer number="16" name="Bottom" color="1" fill="1" visible="yes" active="no"/>
-<layer number="17" name="Pads" color="2" fill="1" visible="yes" active="no"/>
-<layer number="18" name="Vias" color="2" fill="1" visible="yes" active="no"/>
-<layer number="19" name="Unrouted" color="14" fill="1" visible="yes" active="no"/>
-<layer number="20" name="Dimension" color="15" fill="1" visible="yes" active="no"/>
-<layer number="21" name="tPlace" color="7" fill="1" visible="yes" active="no"/>
-<layer number="22" name="bPlace" color="7" fill="1" visible="yes" active="no"/>
-<layer number="23" name="tOrigins" color="15" fill="1" visible="yes" active="no"/>
-<layer number="24" name="bOrigins" color="15" fill="1" visible="yes" active="no"/>
-<layer number="25" name="tNames" color="7" fill="1" visible="yes" active="no"/>
-<layer number="26" name="bNames" color="7" fill="1" visible="yes" active="no"/>
-<layer number="27" name="tValues" color="7" fill="1" visible="yes" active="no"/>
-<layer number="28" name="bValues" color="7" fill="1" visible="yes" active="no"/>
+<layer number="1" name="Top" color="4" fill="1" visible="no" active="no"/>
+<layer number="16" name="Bottom" color="1" fill="1" visible="no" active="no"/>
+<layer number="17" name="Pads" color="2" fill="1" visible="no" active="no"/>
+<layer number="18" name="Vias" color="2" fill="1" visible="no" active="no"/>
+<layer number="19" name="Unrouted" color="14" fill="1" visible="no" active="no"/>
+<layer number="20" name="Dimension" color="15" fill="1" visible="no" active="no"/>
+<layer number="21" name="tPlace" color="7" fill="1" visible="no" active="no"/>
+<layer number="22" name="bPlace" color="7" fill="1" visible="no" active="no"/>
+<layer number="23" name="tOrigins" color="15" fill="1" visible="no" active="no"/>
+<layer number="24" name="bOrigins" color="15" fill="1" visible="no" active="no"/>
+<layer number="25" name="tNames" color="7" fill="1" visible="no" active="no"/>
+<layer number="26" name="bNames" color="7" fill="1" visible="no" active="no"/>
+<layer number="27" name="tValues" color="7" fill="1" visible="no" active="no"/>
+<layer number="28" name="bValues" color="7" fill="1" visible="no" active="no"/>
 <layer number="29" name="tStop" color="7" fill="3" visible="no" active="no"/>
 <layer number="30" name="bStop" color="7" fill="6" visible="no" active="no"/>
@@
 <layer number="35" name="tGlue" color="7" fill="4" visible="no" active="no"/>
 <layer number="36" name="bGlue" color="7" fill="5" visible="no" active="no"/>
-<layer number="37" name="tTest" color="7" fill="1" visible="yes" active="no"/>
-<layer number="38" name="bTest" color="7" fill="1" visible="yes" active="no"/>
+<layer number="37" name="tTest" color="7" fill="1" visible="no" active="no"/>
+<layer number="38" name="bTest" color="7" fill="1" visible="no" active="no"/>
 <layer number="39" name="tKeepout" color="4" fill="11" visible="no" active="no"/>
 <layer number="40" name="bKeepout" color="1" fill="11" visible="no" active="no"/>
@@
 <layer number="44" name="Drills" color="7" fill="1" visible="no" active="no"/>
 <layer number="45" name="Holes" color="7" fill="1" visible="no" active="no"/>
-<layer number="46" name="Milling" color="3" fill="1" visible="yes" active="no"/>
-<layer number="47" name="Measures" color="7" fill="1" visible="yes" active="no"/>
-<layer number="48" name="Document" color="7" fill="1" visible="yes" active="no"/>
-<layer number="49" name="Reference" color="7" fill="1" visible="yes" active="no"/>
-<layer number="50" name="dxf" color="7" fill="1" visible="yes" active="no"/>
-<layer number="51" name="tDocu" color="7" fill="1" visible="yes" active="no"/>
-<layer number="52" name="bDocu" color="7" fill="1" visible="yes" active="no"/>
-<layer number="53" name="tGND_GNDA" color="7" fill="9" visible="yes" active="no"/>
-<layer number="54" name="bGND_GNDA" color="1" fill="9" visible="yes" active="no"/>
-<layer number="56" name="wert" color="7" fill="1" visible="yes" active="no"/>
-<layer number="57" name="tCAD" color="7" fill="1" visible="yes" active="no"/>
-<layer number="59" name="tCarbon" color="7" fill="1" visible="yes" active="no"/>
-<layer number="60" name="bCarbon" color="7" fill="1" visible="yes" active="no"/>
+<layer number="46" name="Milling" color="3" fill="1" visible="no" active="no"/>
+<layer number="47" name="Measures" color="7" fill="1" visible="no" active="no"/>
+<layer number="48" name="Document" color="7" fill="1" visible="no" active="no"/>
+<layer number="49" name="Reference" color="7" fill="1" visible="no" active="no"/>
+<layer number="50" name="dxf" color="7" fill="1" visible="no" active="no"/>
+<layer number="51" name="tDocu" color="7" fill="1" visible="no" active="no"/>
+<layer number="52" name="bDocu" color="7" fill="1" visible="no" active="no"/>
+<layer number="53" name="tGND_GNDA" color="7" fill="9" visible="no" active="no"/>
+<layer number="54" name="bGND_GNDA" color="1" fill="9" visible="no" active="no"/>
+<layer number="56" name="wert" color="7" fill="1" visible="no" active="no"/>
+<layer number="57" name="tCAD" color="7" fill="1" visible="no" active="no"/>
+<layer number="59" name="tCarbon" color="7" fill="1" visible="no" active="no"/>
+<layer number="60" name="bCarbon" color="7" fill="1" visible="no" active="no"/>
 <layer number="90" name="Modules" color="5" fill="1" visible="yes" active="yes"/>
 <layer number="91" name="Nets" color="2" fill="1" visible="yes" active="yes"/>
@@
 <part name="J1" library="SparkFun-Connectors" deviceset="M05" device="JST"/>
 <part name="GND8" library="supply1" deviceset="GND" device=""/>
+<part name="P+8" library="supply1" deviceset="VCC" device=""/>
 </parts>
 <sheets>
@@
 <instance part="J1" gate="G$1" x="33.02" y="81.28"/>
 <instance part="GND8" gate="1" x="45.72" y="68.58"/>
+<instance part="P+8" gate="VCC" x="45.72" y="96.52"/>
 </instances>
 <busses>
@@
 <wire x1="-27.94" y1="55.88" x2="-27.94" y2="66.04" width="0.1524" layer="91"/>
 </segment>
+<segment>
+<pinref part="J1" gate="G$1" pin="5"/>
+<pinref part="P+8" gate="VCC" pin="VCC"/>
+<wire x1="40.64" y1="86.36" x2="45.72" y2="86.36" width="0.1524" layer="91"/>
+<wire x1="45.72" y1="86.36" x2="45.72" y2="93.98" width="0.1524" layer="91"/>
+</segment>
 </net>
 <net name="AREF" class="0">
@@
 <label x="101.6" y="43.18" size="1.27" layer="95" xref="yes"/>
 </segment>
+<segment>
+<pinref part="J1" gate="G$1" pin="4"/>
+<wire x1="48.26" y1="83.82" x2="40.64" y2="83.82" width="0.1524" layer="91"/>
+<label x="48.26" y="83.82" size="1.27" layer="95" xref="yes"/>
+</segment>
 </net>
 <net name="SCL" class="0">
@@
 <label x="101.6" y="40.64" size="1.27" layer="95" xref="yes"/>
 </segment>
-</net>
+<segment>
+<pinref part="J1" gate="G$1" pin="2"/>
+<wire x1="48.26" y1="78.74" x2="40.64" y2="78.74" width="0.1524" layer="91"/>
+<label x="48.26" y="78.74" size="1.27" layer="95" xref="yes"/>
+</segment>
+</net>
